File: pcb/fullScope/fullScope.kicad_pcb (KiCad board)
At the start: 2 copper layers, 92 x 118 mm, 22 parts, among them J1 IN, J2 Conn_02x16_Odd_Even, J3 LCD, J4 Conn_02x18_Odd_Even, J5 Vin, SW1 Btn 1, SW2 Btn 2, SW3 Btn 3, SW4 SW_SPDT, U1 MCP6002-xP, U3 LM7805_TO220

Commit message: fix(pcb): shift J4 to 38.1mm, autoroute traces, update gerbers
Parts:
- moved J4 2.54 mm to (138.1, 100.0)
Routing:
- net CS: track 16.5 -> 8.49 mm
- net RES: track 9.19 -> 16.0 mm
- net GND: track 391.3 -> 385.3 mm
- net BTN2: track 28.0 -> 25.4 mm
- net MOSI: track 8.87 -> 6.33 mm
- net SCK: track 13.6 -> 11.0 mm
- net DC: track 6.65 -> 4.12 mm
- net +3.3V: track 139.0 -> 136.9 mm
- net BTN3: track 28.6 -> 26.6 mm
