File: pcb/fullScope/fullScope.kicad_pcb (KiCad board)
At the start: 2 copper layers, 92 x 118 mm, 22 parts, among them J1 IN, J2 Conn_02x16_Odd_Even, J3 LCD, J4 Conn_02x18_Odd_Even, J5 Vin, SW1 Btn 1, SW2 Btn 2, SW3 Btn 3, SW4 SW_SPDT, U1 MCP6002-xP, U3 LM7805_TO220

Commit message: fix(pcb): update gerber naming extensions, bundle KiCad project zip, and refresh DRC
Co-Authored-By: Claude Code <noreply@anthropic.com>
Parts:
- moved J3 21.0 mm to (162.0, 108.0)
Routing:
- net CS: track 8.49 -> 35.9 mm
- net MOSI: track 6.33 -> 32.3 mm
- net GND: track 385.3 -> 407.7 mm
- net +3.3V: track 136.9 -> 158.4 mm
- net DC: track 4.12 -> 25.1 mm
- net SCK: track 11.0 -> 28.9 mm
- net RES: track 16.0 -> 27.6 mm
